Commit message: added right wheel and joint

File: src/my_robot/urdf/my_robot.xacro (robot description, xacro)
@@ -55,6 +55,5 @@
     </visual>
   </link>
-<link name='left_wheel'>
-    <pose>0 0 0.1 0 0 0</pose>
+    <link name='left_wheel'>
     <inertial>
       <mass value="5.0"/>
@@ -87,3 +86,34 @@
     <dynamics damping="1.0" friction="1.0"/>
   </joint>
+  <link name='right_wheel'>
+    <inertial>
+      <mass value="5.0"/>
+      <origin xyz="0 0 0" rpy=" 0 1.5707 1.5707"/>
+      <inertia
+          ixx="0.1" ixy="0" ixz="0"
+          iyy="0.1" iyz="0"
+          izz="0.1"
+      />
+    </inertial>
+    <collision name='collision'>
+      <origin xyz="0 0 0" rpy=" 0 1.5707 1.5707"/>
+      <geometry>
+        <cylinder radius=".1" length=".05"/>
+      </geometry>
+    </collision>
+    <visual name='right_wheel_visual'>
+      <origin xyz="0 0 0" rpy=" 0 1.5707 1.5707"/>
+      <geometry>
+        <cylinder radius=".1" length=".05"/>
+      </geometry>
+    </visual>
+  </link>
+  <joint type="continuous" name="right_wheel_hinge">
+    <origin xyz="0 -0.15 0" rpy="0 0 0"/>
+    <child link="right_wheel"/>
+    <parent link="chassis"/>
+    <axis xyz="0 -1 0" rpy="0 0 0"/>
+    <limit effort="10000" velocity="1000"/>
+    <dynamics damping="1.0" friction="1.0"/>
+  </joint>
 </robot>

Commit message: added camera and lidar, not working

File: src/my_robot/urdf/my_robot.xacro (robot description, xacro)
@@ -117,3 +117,63 @@
     <dynamics damping="1.0" friction="1.0"/>
   </joint>
+  <!-- Camera -->
+  <link name='camera'>
+    <inertial>
+      <mass value=".1"/>
+      <origin xyz="0 0 0" rpy=" 0 0 0"/>
+      <inertia
+          ixx="1e-6" ixy="0" ixz="0"
+          iyy="1e-6" iyz="0"
+          izz="1e-6"
+      />
+    </inertial>
+    <collision name='collision'>
+      <origin xyz="0 0 0" rpy=" 0 1.5707 1.5707"/>
+      <geometry>
+        <box>
+          <size>.05 .05 .05</size>
+        </box>
+      </geometry>
+    </collision>
+    <visual name='right_wheel_visual'>
+      <origin xyz="0 0 0" rpy=" 0 1.5707 1.5707"/>
+      <geometry>
+        <box>
+          <size>.05 .05 .05</size>
+        </box>
+      </geometry>
+    </visual>
+  </link>
+  <joint type="fixed" name="camera_joint">
+    <origin xyz=".2 0 0" rpy="0 0 0"/>
+    <child link="camera"/>
+    <parent link="chassis"/>
+    <axis xyz="0 1 0" rpy="0 0 0"/>
+  </joint>
+  <!-- Hokuyo Laser -->
+  <link name="hokuyo">
+    <collision>
+      <origin xyz="0 0 0" rpy="0 0 0"/>
+      <geometry>
+	<box size="0.1 0.1 0.1"/>
+      </geometry>
+    </collision>
+    <visual>
+      <origin xyz="0 0 0" rpy="0 0 0"/>
+      <geometry>
+        <mesh filename="package://my_robot/meshes/hokuyo.dae"/>
+      </geometry>
+    </visual>
+    <inertial>
+      <mass value="1e-5" />
+      <origin xyz="0 0 0" rpy="0 0 0"/>
+      <inertia ixx="1e-6" ixy="0" ixz="0" iyy="1e-6" iyz="0" izz="1e-6" />
+    </inertial>
+  </link>
+  <joint name="hokuyo_joint" type="fixed">
+    <axis xyz="0 1 0" />
+    <origin xyz=".15 0 .1 0 0 0" rpy="0 0 0"/>
+    <parent link="chassis"/>
+    <child link="hokuyo"/>
+  </joint>
 </robot>

Commit message: added camera to urdf

File: src/my_robot/urdf/my_robot.xacro (robot description, xacro)
@@ -56,5 +56,5 @@
     </visual>
   </link>
-    <link name='left_wheel'>
+  <link name='left_wheel'>
     <inertial>
       <mass value="5.0"/>
@@ -80,5 +80,5 @@
   </link>
   <joint type="continuous" name="left_wheel_hinge">
-    <origin xyz="0 0.15 0" rpy="0 0 0"/>
+    <origin xyz="0 0.125 0" rpy="0 0 0"/>
     <child link="left_wheel"/>
     <parent link="chassis"/>
@@ -111,5 +111,5 @@
   </link>
   <joint type="continuous" name="right_wheel_hinge">
-    <origin xyz="0 -0.15 0" rpy="0 0 0"/>
+    <origin xyz="0 -0.125 0" rpy="0 0 0"/>
     <child link="right_wheel"/>
     <parent link="chassis"/>
@@ -118,5 +118,5 @@
     <dynamics damping="1.0" friction="1.0"/>
   </joint>
-  <!-- Camera -->
+ <!-- Camera -->
   <link name='camera'>
     <inertial>
@@ -132,7 +132,5 @@
       <origin xyz="0 0 0" rpy=" 0 1.5707 1.5707"/>
       <geometry>
-        <box>
-          <size>.05 .05 .05</size>
-        </box>
+        <box size=".05 .05 .05"/>
       </geometry>
     </collision>
@@ -140,7 +138,5 @@
       <origin xyz="0 0 0" rpy=" 0 1.5707 1.5707"/>
       <geometry>
-        <box>
-          <size>.05 .05 .05</size>
-        </box>
+        <box size=".05 .05 .05"/>
       </geometry>
     </visual>
@@ -163,5 +159,5 @@
       <origin xyz="0 0 0" rpy="0 0 0"/>
       <geometry>
-        <mesh filename="package://my_robot/meshes/hokuyo.dae"/>
+       <box size="0.1 0.1 0.1"/>
       </geometry>
     </visual>
@@ -172,9 +168,9 @@
     </inertial>
   </link>
-  <joint name="hokuyo_joint" type="fixed">
+  <joint type="fixed" name="hokuyo_joint">
+    <origin xyz=".15 0 .1 0 0 0" rpy="0 0 0"/>
+    <child link="hokuyo"/>
+    <parent link="chassis"/>
     <axis xyz="0 1 0" />
-    <origin xyz=".15 0 .1 0 0 0" rpy="0 0 0"/>
-    <parent link="chassis"/>
-    <child link="hokuyo"/>
   </joint>
 </robot>
